Commit message: Add GR3 Mini trajectory tracking task

File: resources/robots/fourier_gr3mini_v200/urdf/gr3mini.urdf (robot description, URDF)
Before this commit: robot gr3miniv2_0_0, 30 links, 29 joints
Links:
- link base_link: geometry collision cylinder length=0.15 radius=0.065; visual mesh filename=../meshes/base_link.STL scale=1 1 1
- link head_pitch_link: geometry collision sphere radius=0.09; visual mesh filename=../meshes/head_pitch_link.STL scale=1 1 1
- link head_yaw_link: geometry visual mesh filename=../meshes/head_yaw_link.STL scale=1 1 1
- link imu_link: geometry visual mesh filename=../meshes/imu_link.STL scale=1 1 1
- link left_foot_pitch_link: geometry visual mesh filename=../meshes/left_foot_pitch_link.STL scale=1 1 1
- link left_foot_roll_link: geometry collision box size=0.205 0.08 0.01; visual mesh filename=../meshes/left_foot_roll_link.STL scale=1 1 1
- link left_hand_yaw_link: geometry collision sphere radius=0.025; visual mesh filename=../meshes/left_hand_yaw_link.STL scale=1 1 1
- link left_lower_arm_pitch_link: geometry collision cylinder length=0.09 radius=0.034; visual mesh filename=../meshes/left_lower_arm_pitch_link.STL scale=1 1 1
- link left_shank_pitch_link: geometry collision cylinder length=0.2 radius=0.06; visual mesh filename=../meshes/left_shank_pitch_link.STL scale=1 1 1
- link left_thigh_pitch_link: geometry visual mesh filename=../meshes/left_thigh_pitch_link.STL scale=1 1 1
- link left_thigh_roll_link: geometry visual mesh filename=../meshes/left_thigh_roll_link.STL scale=1 1 1
- link left_thigh_yaw_link: geometry collision cylinder length=0.16 radius=0.045; visual mesh filename=../meshes/left_thigh_yaw_link.STL scale=1 1 1
- link left_upper_arm_pitch_link: geometry visual mesh filename=../meshes/left_upper_arm_pitch_link.STL scale=1 1 1
- link left_upper_arm_roll_link: geometry collision cylinder length=0.08 radius=0.035; visual mesh filename=../meshes/left_upper_arm_roll_link.STL scale=1 1 1
- link left_upper_arm_yaw_link: geometry collision cylinder length=0.08 radius=0.03; collision cylinder length=0.08 radius=0.038
- link right_foot_pitch_link: geometry visual mesh filename=../meshes/right_foot_pitch_link.STL scale=1 1 1
- link right_foot_roll_link: geometry collision box size=0.205 0.08 0.01; visual mesh filename=../meshes/right_foot_roll_link.STL scale=1 1 1
- link right_hand_yaw_link: geometry collision sphere radius=0.025; visual mesh filename=../meshes/left_hand_yaw_link.STL scale=1 1 1
- link right_lower_arm_pitch_link: geometry collision cylinder length=0.09 radius=0.034; visual mesh filename=../meshes/right_lower_arm_pitch_link.STL scale=1 1 1
- link right_shank_pitch_link: geometry collision cylinder length=0.2 radius=0.06; visual mesh filename=../meshes/right_shank_pitch_link.STL scale=1 1 1
- link right_thigh_pitch_link: geometry visual mesh filename=../meshes/right_thigh_pitch_link.STL scale=1 1 1
- link right_thigh_roll_link: geometry visual mesh filename=../meshes/right_thigh_roll_link.STL scale=1 1 1
- link right_thigh_yaw_link: geometry collision cylinder length=0.16 radius=0.045; visual mesh filename=../meshes/right_thigh_yaw_link.STL scale=1 1 1
- link right_upper_arm_pitch_link: geometry visual mesh filename=../meshes/right_upper_arm_pitch_link.STL scale=1 1 1
- link right_upper_arm_roll_link: geometry collision cylinder length=0.08 radius=0.035; visual mesh filename=../meshes/right_upper_arm_roll_link.STL scale=1 1 1
- link right_upper_arm_yaw_link: geometry collision cylinder length=0.08 radius=0.03; collision cylinder length=0.08 radius=0.038
- link torso_link: geometry collision box size=0.2 0.15 0.25; visual mesh filename=../meshes/torso_link.STL scale=1 1 1
- link waist_yaw_link: geometry visual mesh filename=../meshes/waist_yaw_link.STL scale=1 1 1
Joints:
- removed joint left_wrist_yaw_joint 
- removed joint right_wrist_yaw_joint 
- added joint left_wrist_yaw_joint: type revolute, parent left_lower_arm_pitch_link, child left_hand_yaw_link, origin xyz=-0.02 -0.022 -0.135 rpy=0 0 0, axis 0.0 0.0 1.0, limit lower=-1.4835 upper=1.4835 effort=11.0 velocity=5.233
- added joint right_wrist_yaw_joint: type revolute, parent right_lower_arm_pitch_link, child right_hand_yaw_link, origin xyz=-0.02 0.022 -0.135 rpy=0 0 0, axis 0.0 0.0 1.0, limit lower=-1.4835 upper=1.4835 effort=11.0 velocity=5.233
